Commit message: added robot base added path constraints

File: config/gazebo_ur5e.urdf (robot description, URDF)
Before this commit: robot ur5e, 27 links, 26 joints
Links:
- added link robot_base_column, mass 0.1; collision box size=0.15 0.15 0.44; visual box size=0.15 0.15 0.44
- added link robot_base_table, mass 0.1; collision box size=0.6 0.6 0.02; visual box size=0.6 0.6 0.02
- added link safety_wall, mass 0.1; collision box size=3 0.1 3; visual box size=3 0.1 3
- added link table, mass 0.1; collision box size=3 3 0.001; visual box size=3 3 0.001
- link onrobot_link: mass 1 -> 0.1
Joints:
- added joint robot_base_column_table: type fixed, parent robot_base_column, child table, origin xyz=2 -0.15 0.02 rpy=0 0 0
- added joint robot_base_table_column: type fixed, parent robot_base_table, child robot_base_column, origin xyz=0 0 0.22 rpy=0 0 0
- added joint safety_wall_base_link: type fixed, parent safety_wall, child base_link, origin xyz=0.0 -0.4 0.0 rpy=0 0 0
- added joint table_safety_wall: type fixed, parent table, child safety_wall, origin xyz=-2 0.55 0.2 rpy=0 0 0
- joint gripper_joint: origin xyz=0 0 0.07835 rpy=1.57 0 0 -> xyz=0 0 0.07835 rpy=1.57 0 2.355
